File: hardware/crackedbadusb.kicad_sch (KiCad schematic)
At the start: 38 parts, among them Q1 AO3400A_C347475, Q2 XC6220B331MR-G, U1 RP2040, U2 DSHP04TSGER_C3293144, U3 USBLC6-2SC6, U4 W25Q128JVS, U5 ABM8-272-T3_C20625731, U8 Ai-Thinker-Ra-02

Commit message: blueprint compliance stuff
Other:
- title: crackedbadusb (crb) -> scriptstick (previously called crackedbadusb)
Changed lines of the file:
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@@
 	(paper "A4")
 	(title_block
-		(title "crackedbadusb (crb)")
+		(title "scriptstick (previously called crackedbadusb)")
 		(date "2025-11-05")
 		(rev "1.0")
@@
 	)
 	(no_connect
-		(at 190.5 133.35)
+		(at 166.37 92.71)
 	)
 	(no_connect
@@
 	)
 	(no_connect
-		(at 190.5 128.27)
+		(at 166.37 87.63)
 	)
 	(no_connect
@@
 	)
 	(no_connect
-		(at 190.5 130.81)
+		(at 166.37 90.17)
 	)
 	(no_connect
@@
 	)
 	(no_connect
-		(at 190.5 135.89)
+		(at 166.37 95.25)
 	)
 	(no_connect
@@
 	(wire
 		(pts
-			(xy 184.15 130.81) (xy 190.5 130.81)
-		)
-		(stroke
-			(width 0)
-			(type default)
-		)
-	)
-	(wire
-		(pts
 			(xy 222.25 110.49) (xy 222.25 67.31)
 		)
@@
 	(wire
 		(pts
-			(xy 181.61 135.89) (xy 181.61 95.25)
-		)
-		(stroke
-			(width 0)
-			(type default)
-		)
-	)
-	(wire
-		(pts
 			(xy 92.71 85.09) (xy 92.71 82.55)
 		)
@@
 	(wire
 		(pts
-			(xy 166.37 90.17) (xy 184.15 90.17)
-		)
-		(stroke
-			(width 0)
-			(type default)
-		)
-	)
-	(wire
-		(pts
 			(xy 115.57 87.63) (xy 95.25 87.63)
 		)
@@
 	(wire
 		(pts
-			(xy 182.88 92.71) (xy 166.37 92.71)
-		)
-		(stroke
-			(width 0)
-			(type default)
-		)
-	)
-	(wire
-		(pts
 			(xy 160.02 34.29) (xy 171.45 34.29)
 		)
@@
 	(wire
 		(pts
-			(xy 185.42 87.63) (xy 166.37 87.63)
-		)
-		(stroke
-			(width 0)
-			(type default)
-		)
-	)
-	(wire
-		(pts
-			(xy 182.88 133.35) (xy 182.88 92.71)
-		)
-		(stroke
-			(width 0)
-			(type default)
-		)
-	)
-	(wire
-		(pts
 			(xy 54.61 157.48) (xy 63.5 157.48)
 		)
@@
 	(wire
 		(pts
-			(xy 190.5 128.27) (xy 185.42 128.27)
-		)
-		(stroke
-			(width 0)
-			(type default)
-		)
-	)
-	(wire
-		(pts
 			(xy 93.98 120.65) (xy 93.98 118.11)
 		)
@@
 	(wire
 		(pts
-			(xy 184.15 90.17) (xy 184.15 130.81)
-		)
-		(stroke
-			(width 0)
-			(type default)
-		)
-	)
-	(wire
-		(pts
 			(xy 273.05 40.64) (xy 271.78 40.64)
 		)
@@
 	(wire
 		(pts
-			(xy 181.61 95.25) (xy 166.37 95.25)
-		)
-		(stroke
-			(width 0)
-			(type default)
-		)
-	)
-	(wire
-		(pts
 			(xy 166.37 125.73) (xy 168.91 125.73)
 		)
@@
 	(wire
 		(pts
-			(xy 185.42 128.27) (xy 185.42 87.63)
-		)
-		(stroke
-			(width 0)
-			(type default)
-		)
-	)
-	(wire
-		(pts
 			(xy 135.89 49.53) (xy 138.43 49.53)
 		)
@@
 	(wire
 		(pts
-			(xy 190.5 135.89) (xy 181.61 135.89)
-		)
-		(stroke
-			(width 0)
-			(type default)
-		)
-	)
-	(wire
-		(pts
 			(xy 25.4 156.21) (xy 17.78 156.21)
 		)
@@
 		)
 		(stroke
-			(width 0)
-			(type default)
-		)
-	)
-	(wire
-		(pts
-			(xy 190.5 133.35) (xy 182.88 133.35)
-		)
-		(stroke
